File: Hardware/LED Cube.sch (EAGLE design)
At the start: 223 parts, among them IC1 MEGA8-AI, IC10 FT232RL, IC11 FM24V10, IC12 MSGEQ7, IC14 MEGA32-A, IC2 74HC573D, IC3 74HC573D, IC4 74HC573D, IC5 74HC573D, IC6 74HC573D, IC7 74HC573D, IC8 74HC573D, IC9 74HC573D, X2 USB-B-MINI-SMD

Commit message: Ordered PCB
Parts:
- C19, C20, C22, C23, C24, C25, C26, C27, C28, C29, C30: value (none) -> 100n
- C21: value (none) -> 4u7
Changed lines of the file:
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@@
 <part name="GND38" library="supply1" deviceset="GND" device=""/>
 <part name="P+10" library="supply1" deviceset="VCC" device=""/>
-<part name="C19" library="resistor" deviceset="C-EU" device="C0603"/>
-<part name="C20" library="resistor" deviceset="C-EU" device="C0603"/>
-<part name="C21" library="resistor" deviceset="CPOL-EU" device="TAP5-80"/>
+<part name="C19" library="resistor" deviceset="C-EU" device="C0603" value="100n"/>
+<part name="C20" library="resistor" deviceset="C-EU" device="C0603" value="100n"/>
+<part name="C21" library="resistor" deviceset="CPOL-EU" device="TAP5-80" value="4u7"/>
 <part name="JP2" library="jumper" deviceset="JP1E" device=""/>
 <part name="X1" library="con-conrad" deviceset="73398?" device="0-62"/>
-<part name="C22" library="resistor" deviceset="C-EU" device="C0603"/>
-<part name="C23" library="resistor" deviceset="C-EU" device="C0603"/>
-<part name="C24" library="resistor" deviceset="C-EU" device="C0603"/>
-<part name="C25" library="resistor" deviceset="C-EU" device="C0603"/>
-<part name="C26" library="resistor" deviceset="C-EU" device="C0603"/>
-<part name="C27" library="resistor" deviceset="C-EU" device="C0603"/>
-<part name="C28" library="resistor" deviceset="C-EU" device="C0603"/>
-<part name="C29" library="resistor" deviceset="C-EU" device="C0603"/>
-<part name="C30" library="resistor" deviceset="C-EU" device="C0603"/>
+<part name="C22" library="resistor" deviceset="C-EU" device="C0603" value="100n"/>
+<part name="C23" library="resistor" deviceset="C-EU" device="C0603" value="100n"/>
+<part name="C24" library="resistor" deviceset="C-EU" device="C0603" value="100n"/>
+<part name="C25" library="resistor" deviceset="C-EU" device="C0603" value="100n"/>
+<part name="C26" library="resistor" deviceset="C-EU" device="C0603" value="100n"/>
+<part name="C27" library="resistor" deviceset="C-EU" device="C0603" value="100n"/>
+<part name="C28" library="resistor" deviceset="C-EU" device="C0603" value="100n"/>
+<part name="C29" library="resistor" deviceset="C-EU" device="C0603" value="100n"/>
+<part name="C30" library="resistor" deviceset="C-EU" device="C0603" value="100n"/>
 <part name="P+80" library="supply1" deviceset="VCC" device=""/>
 <part name="GND40" library="supply1" deviceset="GND" device=""/>
