File: Hardware/LED Cube.brd (EAGLE design)
At the start: 160 x 100 mm, 210 parts, among them IC1 MEGA8-AI, IC10 FT232RL, IC11 FM24V10, IC12 MSGEQ7, IC14 MEGA32-A, IC2 74HC573D, IC3 74HC573D, IC4 74HC573D, IC5 74HC573D, IC6 74HC573D, IC7 74HC573D, IC8 74HC573D, IC9 74HC573D

Commit message: Worked at Layout
Parts:
- removed R22: (no value), resistor:RTRIM3296W
- removed S1: (no value), switch:255SB
- removed V1: 7400N, 74ttl-din:DIL14
- added U$74: TASTER, 0-xythobuz:SMDTASTER
- R18: value 1k -> (none); device resistor:R0603 -> pot:PT-10S
- moved R86 248.1 mm to (129.1, 84.4), turned to 180 degrees
- moved R85 243.3 mm to (129.1, 82.3), turned to 180 degrees
- moved R62 242.5 mm to (129.1, 47.5), turned to 180 degrees
- moved U$9 241.7 mm to (98.2, 23.3)
- moved U$8 241.4 mm to (103.8, 25.2)
- moved R84 238.4 mm to (129.2, 80.1), turned to 180 degrees
- moved R61 238.1 mm to (129.1, 45.4), turned to 180 degrees
- moved R83 234.3 mm to (129.3, 73.8), turned to 180 degrees
- moved R60 233.6 mm to (129.1, 43.3), turned to 180 degrees
- moved U$31 233.6 mm to (98.2, 48.8)
- moved U$30 232.0 mm to (103.8, 55.1)
- moved U$7 230.6 mm to (98.1, 27.6)
- moved R59 230.2 mm to (129.0, 37.0), turned to 180 degrees
- moved R82 229.6 mm to (129.3, 71.7), turned to 180 degrees
- moved U$6 228.7 mm to (103.7, 33.6)
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Connections:
- removed net N$72: V1.2, V1.6
- removed net N$73: R18.1, S1.3, V1.5
- removed net N$74: R20.2, S1.1, V1.1
- net GND: now also R18.E, U$74.B, U$74.B2; no longer R22.3, S1.2, V1.7
- net N$69: now also R20.2, U$74.A, U$74.A2; no longer V1.3, V1.4
- net N$77: now also R18.S; no longer R22.2
- net VCC: now also R18.A; no longer R18.2, R22.1, V1.14
Routing:
- net VCC: track 37.8 -> 605.2 mm, vias 8 -> 65
- net N$13: track 0.00 -> 439.2 mm, vias 0 -> 14
- net N$11: track 0.00 -> 404.5 mm, vias 0 -> 16
- net N$9: track 0.00 -> 401.1 mm, vias 0 -> 14
- net N$12: track 0.00 -> 401.0 mm, vias 0 -> 15
- net N$5: track 0.00 -> 368.0 mm, vias 0 -> 16
- net N$10: track 0.00 -> 367.0 mm, vias 0 -> 14
- net N$6: track 0.00 -> 360.7 mm, vias 0 -> 15
- net N$4: track 0.00 -> 354.6 mm, vias 0 -> 13
- net GND: track 0.00 -> 194.4 mm, vias 0 -> 23
- net N$51: track 0.00 -> 62.5 mm
- net N$50: track 0.00 -> 60.6 mm, vias 0 -> 2
- net N$57: track 0.00 -> 56.1 mm, vias 0 -> 2
- net N$53: track 0.00 -> 52.9 mm
- net N$69: track 0.00 -> 50.3 mm, vias 0 -> 2
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- added copper zone on layer 1, net N$40
Other:
- board text added: "CubeControl"

Commit message: Finished Layout
Parts:
- added C19, C20, C22, C23, C24, C25, C26, C27, C28, C29, C30: (no value), resistor:C0603
- added C21: (no value), resistor:TAP5-80
- added IC13: (no value), v-reg:78XXS
- added JP2: (no value), jumper:JP1
- added X1: (no value), con-conrad:733980-62
- moved C13 19.9 mm to (26.9, 1.91)
- moved U$1 17.8 mm to (-0.11, 0.77)
- moved R17 13.7 mm to (16.3, 4.21)
- moved R16 12.9 mm to (16.3, 1.71)
- moved JP6 9.90 mm to (57.3, 4.71)
- moved R19 9.90 mm to (45.0, 4.69)
- moved IC11 2.10 mm to (47.5, 58.0)
- moved R14 2.10 mm to (48.5, 65.7)
- moved U$74 1.08 mm to (63.1, 51.2)
- moved LED1 0.71 mm to (51.6, 16.4)
- moved LED65 0.71 mm to (53.2, 16.4)
- moved R31 0.71 mm to (51.3, 12.2)
- moved R21 0.71 mm to (53.5, 12.2)
- moved U$15 0.20 mm to (120.7, 26.6)
- moved R47 0.10 mm to (129.2, 15.8)
Connections:
- new net N$74: C20.1, C21.+, IC13.IN, X1.2
- new net N$84: C19.1, IC13.OUT, JP2.1
- net GND: now also C19.2, C20.2, C21.-, C22.1, C23.1, C24.1, C25.1, C26.1, C27.1, C28.1, C29.1, C30.1, IC13.GND, X1.1
- net VCC: now also C22.2, C23.2, C24.2, C25.2, C26.2, C27.2, C28.2, C29.2, C30.2, JP2.2
Routing:
- net VCC: track 605.2 -> 966.5 mm, vias 65 -> 69
- net N$16: track 0.00 -> 229.9 mm, vias 0 -> 6
- net N$17: track 0.00 -> 214.3 mm, vias 0 -> 6
- net N$19: track 0.00 -> 203.2 mm, vias 0 -> 6
- net N$20: track 0.00 -> 174.3 mm, vias 0 -> 4
- net GND: track 194.4 -> 344.1 mm, vias 23 -> 35
- net N$30: track 0.00 -> 123.9 mm, vias 0 -> 2
- net N$29: track 0.00 -> 111.1 mm, vias 0 -> 2
- net N$21: track 0.00 -> 87.6 mm, vias 0 -> 4
- net N$65: track 0.00 -> 73.3 mm, vias 0 -> 1
- net N$15: track 0.00 -> 69.0 mm, vias 0 -> 4
- net N$67: track 0.00 -> 65.9 mm, vias 0 -> 1
- net N$18: track 0.00 -> 62.0 mm, vias 0 -> 4
- net N$14: track 0.00 -> 51.8 mm, vias 0 -> 4
- net N$68: track 0.00 -> 49.8 mm, vias 0 -> 1
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
Commit message: Ordered PCB
Parts:
- C19, C20, C22, C23, C24, C25, C26, C27, C28, C29, C30: value (none) -> 100n
- C21: value (none) -> 4u7
Routing:
- net VCC: track 966.5 -> 968.8 mm
- added copper zone on layer 1, net GND
- removed copper zone on layer 1, net N$40
Other:
- board text added: "12V"
- board text added: "BOTTOM"
- board text added: "ISP 1"
- board text added: "ISP 2"
- board text added: "LAYER"
- board text added: "LED Cube"
- board text added: "PC"
- board text added: "TOP"
- board text added: "www.xythobuz.org"
- board text removed: "CubeControl"
Changed lines of the file:
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@@
 <layer number="21" name="tPlace" color="7" fill="1" visible="yes" active="yes"/>
 <layer number="22" name="bPlace" color="7" fill="1" visible="yes" active="yes"/>
-<layer number="23" name="tOrigins" color="15" fill="1" visible="yes" active="yes"/>
-<layer number="24" name="bOrigins" color="15" fill="1" visible="yes" active="yes"/>
-<layer number="25" name="tNames" color="7" fill="1" visible="yes" active="yes"/>
-<layer number="26" name="bNames" color="7" fill="1" visible="yes" active="yes"/>
+<layer number="23" name="tOrigins" color="15" fill="1" visible="no" active="yes"/>
+<layer number="24" name="bOrigins" color="15" fill="1" visible="no" active="yes"/>
+<layer number="25" name="tNames" color="7" fill="1" visible="no" active="yes"/>
+<layer number="26" name="bNames" color="7" fill="1" visible="no" active="yes"/>
 <layer number="27" name="tValues" color="7" fill="1" visible="no" active="yes"/>
-<layer number="28" name="bValues" color="7" fill="1" visible="yes" active="yes"/>
+<layer number="28" name="bValues" color="7" fill="1" visible="no" active="yes"/>
 <layer number="29" name="tStop" color="7" fill="3" visible="no" active="yes"/>
 <layer number="30" name="bStop" color="7" fill="6" visible="no" active="yes"/>
@@
 <wire x1="160" y1="100" x2="0" y2="100" width="0" layer="20"/>
 <wire x1="0" y1="100" x2="0" y2="0" width="0" layer="20"/>
-<text x="122" y="90.9" size="3.81" layer="1" font="vector">CubeControl</text>
+<text x="156.6" y="90.3" size="5.08" layer="16" font="vector" rot="MR0">LED Cube</text>
+<text x="158.2" y="2.8" size="2.54" layer="16" font="vector" rot="MR0">www.xythobuz.org</text>
+<text x="124.6" y="2" size="2.54" layer="1" font="vector">www.xythobuz.org</text>
+<text x="49.8" y="95.2" size="2.54" layer="1" font="vector">TOP</text>
+<text x="59.3" y="95.3" size="2.54" layer="16" font="vector" rot="MR0">BOTTOM</text>
+<text x="121.3" y="90.3" size="5.08" layer="1" font="vector">LED Cube</text>
+<text x="68.7" y="1.5" size="2.54" layer="1" font="vector">ISP 2</text>
+<text x="11.8" y="96.7" size="2.54" layer="1" font="vector">ISP 1</text>
+<text x="1.5" y="85" size="2.54" layer="1" font="vector">PC</text>
+<text x="1.3" y="64.3" size="2.54" layer="1" font="vector">LAYER</text>
+<text x="13.9" y="20.5" size="2.54" layer="1" font="vector">12V</text>
 </plain>
 <attributes>
@@
 <param name="rvMicroViaOuter" value="0.25"/>
 <param name="rvMicroViaInner" value="0.25"/>
-<param name="rlMinPadTop" value="10mil"/>
+<param name="rlMinPadTop" value="0.15mm"/>
 <param name="rlMaxPadTop" value="20mil"/>
-<param name="rlMinPadInner" value="10mil"/>
+<param name="rlMinPadInner" value="0.15mm"/>
 <param name="rlMaxPadInner" value="20mil"/>
-<param name="rlMinPadBottom" value="10mil"/>
+<param name="rlMinPadBottom" value="0.15mm"/>
 <param name="rlMaxPadBottom" value="20mil"/>
-<param name="rlMinViaOuter" value="8mil"/>
+<param name="rlMinViaOuter" value="0.15mm"/>
 <param name="rlMaxViaOuter" value="20mil"/>
-<param name="rlMinViaInner" value="8mil"/>
+<param name="rlMinViaInner" value="0.15mm"/>
 <param name="rlMaxViaInner" value="20mil"/>
-<param name="rlMinMicroViaOuter" value="4mil"/>
+<param name="rlMinMicroViaOuter" value="0.15mm"/>
 <param name="rlMaxMicroViaOuter" value="20mil"/>
-<param name="rlMinMicroViaInner" value="4mil"/>
+<param name="rlMinMicroViaInner" value="0.15mm"/>
 <param name="rlMaxMicroViaInner" value="20mil"/>
 <param name="psTop" value="-1"/>
@@
 <param name="checkFont" value="1"/>
 <param name="checkRestrict" value="1"/>
-<param name="useDiameter" value="13"/>
+<param name="useDiameter" value="31"/>
 <param name="maxErrors" value="50"/>
 </designrules>
@@
 <element name="R18" library="pot" package="PT-10S" value="" x="63.4" y="15.9" rot="R90"/>
 <element name="IC13" library="v-reg" package="78XXS" value="" x="-0.7" y="32.7" rot="R90"/>
-<element name="C19" library="resistor" package="C0603" value="" x="5.4" y="35.7" rot="R270"/>
-<element name="C20" library="resistor" package="C0603" value="" x="5.2" y="30.5" rot="R90"/>
-<element name="C21" library="resistor" package="TAP5-80" value="" x="11.6" y="30.5" rot="R90"/>
+<element name="C19" library="resistor" package="C0603" value="100n" x="5.4" y="35.7" rot="R270"/>
+<element name="C20" library="resistor" package="C0603" value="100n" x="5.2" y="30.5" rot="R90"/>
+<element name="C21" library="resistor" package="TAP5-80" value="4u7" x="11.6" y="30.5" rot="R90"/>
 <element name="JP2" library="jumper" package="JP1" value="" x="6.7" y="40.5" rot="R270"/>
 <element name="X1" library="con-conrad" package="733980-62" value="" x="2.6" y="21.7" rot="R270"/>
-<element name="C22" library="resistor" package="C0603" value="" x="45.6" y="59.6" rot="R90"/>
-<element name="C23" library="resistor" package="C0603" value="" x="81.5" y="82.9"/>
-<element name="C24" library="resistor" package="C0603" value="" x="81.2" y="65.1"/>
-<element name="C25" library="resistor" package="C0603" value="" x="81.2" y="44"/>
-<element name="C26" library="resistor" package="C0603" value="" x="81.4" y="22.7"/>
-<element name="C27" library="resistor" package="C0603" value="" x="139.6" y="15.7" rot="R180"/>
-<element name="C28" library="resistor" package="C0603" value="" x="139.7" y="32.6" rot="R180"/>
-<element name="C29" library="resistor" package="C0603" value="" x="139.7" y="51" rot="R180"/>
-<element name="C30" library="resistor" package="C0603" value="" x="139.8" y="68.2" rot="R180"/>
+<element name="C22" library="resistor" package="C0603" value="100n" x="45.6" y="59.6" rot="R90"/>
+<element name="C23" library="resistor" package="C0603" value="100n" x="81.5" y="82.9"/>
+<element name="C24" library="resistor" package="C0603" value="100n" x="81.2" y="65.1"/>
+<element name="C25" library="resistor" package="C0603" value="100n" x="81.2" y="44"/>
+<element name="C26" library="resistor" package="C0603" value="100n" x="81.4" y="22.7"/>
+<element name="C27" library="resistor" package="C0603" value="100n" x="139.6" y="15.7" rot="R180"/>
+<element name="C28" library="resistor" package="C0603" value="100n" x="139.7" y="32.6" rot="R180"/>
+<element name="C29" library="resistor" package="C0603" value="100n" x="139.7" y="51" rot="R180"/>
+<element name="C30" library="resistor" package="C0603" value="100n" x="139.8" y="68.2" rot="R180"/>
 </elements>
 <signals>
@@
 <contactref element="U$72" pad="3"/>
 <contactref element="U$73" pad="3"/>
-<polygon width="0.4064" layer="16" isolate="0.35">
+<polygon width="0.4064" layer="16" isolate="0.4">
 <vertex x="0" y="0"/>
 <vertex x="160" y="0"/>
@@
 <via x="53.6" y="23.7" extent="1-16" drill="0.4"/>
 <wire x1="53.6" y1="23.7" x2="53.6" y2="24" width="0.4064" layer="16"/>
+<polygon width="0.4064" layer="1" isolate="0.4">
+<vertex x="0" y="0"/>
+<vertex x="160" y="0"/>
+<vertex x="160" y="100"/>
+<vertex x="0" y="100"/>
+</polygon>
 </signal>
 <signal name="VCC">
@@
 <wire x1="120.09" y1="27.25" x2="119.85" y2="27.25" width="0.4064" layer="1"/>
 <wire x1="119.85" y1="27.25" x2="119.3" y2="27.8" width="0.4064" layer="1"/>
-<wire x1="21.44" y1="72.91" x2="21.38" y2="70.71" width="0" layer="19" extent="1-1"/>
+<wire x1="21.44" y1="72.91" x2="21.38" y2="72.91" width="0.4064" layer="1"/>
+<wire x1="21.38" y1="72.91" x2="21.38" y2="70.71" width="0.4064" layer="1"/>
 </signal>
 <signal name="N$2">
@@
 <wire x1="80.275" y1="49.375" x2="80.3" y2="49.4" width="0.4064" layer="1"/>
 <via x="80.3" y="49.4" extent="1-16" drill="0.4"/>
-<wire x1="80.3" y1="49.4" x2="66.8" y2="49.4" width="0.4064" layer="16"/>
-<wire x1="66.8" y1="49.4" x2="66.6" y2="49.2" width="0.4064" layer="16"/>
 <via x="66.6" y="49.3" extent="1-16" drill="0.4"/>
 <wire x1="66.6" y1="49.3" x2="66.6" y2="69.7" width="0.4064" layer="1"/>
@@
 <wire x1="155.6" y1="27" x2="155.6" y2="26.9" width="0.4064" layer="16"/>
 <via x="155.6" y="26.9" extent="1-16" drill="0.4"/>
-<wire x1="66.6" y1="49.3" x2="66.6" y2="49.2" width="0" layer="19" extent="16-16"/>
+<wire x1="80.3" y1="49.4" x2="66.6" y2="49.4" width="0.4064" layer="16"/>
+<wire x1="66.6" y1="49.4" x2="66.6" y2="49.3" width="0.4064" layer="16"/>
 </signal>
 <signal name="N$13">
@@
 <wire x1="12.2" y1="59.5" x2="16.6" y2="59.5" width="0.4064" layer="16"/>
 </signal>
-<signal name="N$40">
-<polygon width="0.4064" layer="1" isolate="0.5">
-<vertex x="120" y="89.1"/>
-<vertex x="158.2" y="89.1"/>
-<vertex x="158.2" y="96.4"/>
-<vertex x="120" y="96.4"/>
-</polygon>
-</signal>
 <signal name="N$74">
 <contactref element="C21" pad="+"/>
@@
 </signal>
 </signals>
-<errors>
-</errors>
 </board>
 </drawing>
